File: selector.kicad_pcb (KiCad board)
At the start: 2 copper layers, 35 x 110 mm, 31 parts, among them J1 Conn_02x05_Odd_Even, SW1 PEC11R, U1 TLC5916, U2 TLC5916

Commit message: Adds Front Panel
Other:
- board text added: "Selector Board"
- board text removed: "Spud Board"
Changed lines of the file:
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@@
     (tags "mounting hole 3.2mm no annular m3")
     (attr virtual)
-    (fp_text reference H1 (at 4.5 -2) (layer F.SilkS)
+    (fp_text reference H1 (at 0 0) (layer F.SilkS)
       (effects (font (size 1 1) (thickness 0.15)))
     )
@@
     (tags "mounting hole 3.2mm no annular m3")
     (attr virtual)
-    (fp_text reference H2 (at -4.5 -2.5) (layer F.SilkS)
+    (fp_text reference H2 (at 0 0) (layer F.SilkS)
       (effects (font (size 1 1) (thickness 0.15)))
     )
@@
     (tags "mounting hole 3.2mm no annular m3")
     (attr virtual)
-    (fp_text reference H3 (at 0 -4.2) (layer F.SilkS)
+    (fp_text reference H3 (at 0 0) (layer F.SilkS)
       (effects (font (size 1 1) (thickness 0.15)))
     )
@@
     (tags "mounting hole 3.2mm no annular m3")
     (attr virtual)
-    (fp_text reference H4 (at 0 -4.2) (layer F.SilkS)
+    (fp_text reference H4 (at 0 0) (layer F.SilkS)
       (effects (font (size 1 1) (thickness 0.15)))
     )
@@
     (effects (font (size 1.5 1.5) (thickness 0.15)))
   )
-  (gr_text "Spud Board" (at 77.5 67.5) (layer F.SilkS)
+  (gr_text "Selector Board" (at 77.5 67.5) (layer F.SilkS)
     (effects (font (size 2 2) (thickness 0.15)))
   )

Commit message: Latest changes.
Parts:
- C4: value 100uF -> 47uF; footprint Capacitor_THT:CP_Radial_D8.0mm_P3.50mm -> Capacitor_THT:CP_Radial_D6.3mm_P2.50mm
- moved C4 0.50 mm to (87.5, 106.0)
Connections:
- J1 pad 7: Net-(J1-Pad7) -> Net-(C2-Pad1)
- J1 pad 8: Net-(J1-Pad8) -> Net-(C1-Pad1)
- R1 pad 1: Net-(J1-Pad8) -> Net-(C1-Pad1)
- R1 pad 2: Net-(C1-Pad1) -> Net-(R1-Pad2)
- R2 pad 1: Net-(J1-Pad7) -> Net-(C2-Pad1)
- R2 pad 2: Net-(C2-Pad1) -> Net-(R2-Pad2)
- R3 pad 2: Net-(C1-Pad1) -> Net-(R1-Pad2)
- R5 pad 2: Net-(C2-Pad1) -> Net-(R2-Pad2)
- SW1 pad A: Net-(C1-Pad1) -> Net-(R1-Pad2)
- SW1 pad B: Net-(C2-Pad1) -> Net-(R2-Pad2)
Routing:
- net Net-(J1-Pad8): track 51.1 -> 0.00 mm, vias 2 -> 0
- net Net-(J1-Pad7): track 46.3 -> 0.00 mm
- net Net-(C1-Pad1): track 33.5 -> 77.0 mm, vias 0 -> 2
- net Net-(C2-Pad1): track 28.0 -> 69.1 mm
- net Net-(R2-Pad2): track 0.00 -> 25.9 mm
- net Net-(R1-Pad2): track 0.00 -> 25.1 mm
- net GND: track 14.7 -> 0.00 mm
- net Net-(J1-Pad9): track 59.7 -> 58.9 mm

Commit message: Update
Parts:
- added R7: 1K, Resistor_THT:R_Axial_DIN0207_L6.3mm_D2.5mm_P10.16mm_Horizontal, F.Cu at (82.4, 132.0)
- R4, R6: value 2K -> 2.2K
- moved C5 2.50 mm to (79.5, 75.0)
Connections:
- SW1 pad 2: Net-(J1-Pad9) -> Net-(R7-Pad1)
Routing:
- net Net-(J1-Pad9): track 58.9 -> 34.7 mm
- net Net-(R7-Pad1): track 0.00 -> 19.9 mm
- net Net-(C2-Pad1): track 69.1 -> 74.6 mm, vias 0 -> 1
Other:
- board text added: "v1.2"
- board text removed: "v1.1"
Changed lines of the file:
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@@
     (thickness 1.6)
     (drawings 7)
-    (tracks 155)
+    (tracks 160)
     (zones 0)
-    (modules 31)
-    (nets 32)
+    (modules 32)
+    (nets 33)
   )
   (page A4)
@@
   (net 30 "Net-(R1-Pad2)")
   (net 31 "Net-(R2-Pad2)")
+  (net 32 "Net-(R7-Pad1)")
   (net_class Default "This is the default net class."
     (clearance 0.2)
@@
     (add_net "Net-(R4-Pad1)")
     (add_net "Net-(R6-Pad1)")
+    (add_net "Net-(R7-Pad1)")
     (add_net "Net-(U1-Pad14)")
     (add_net "Net-(U2-Pad10)")
@@
       (effects (font (size 1 1) (thickness 0.15)))
     )
-    (fp_text value 2K (at 5.08 2.37 90) (layer F.Fab)
+    (fp_text value 2.2K (at 5.08 2.37 90) (layer F.Fab)
       (effects (font (size 1 1) (thickness 0.15)))
     )
@@
       (effects (font (size 1 1) (thickness 0.15)))
     )
-    (fp_text value 2K (at 5.08 2.37 90) (layer F.Fab)
+    (fp_text value 2.2K (at 5.08 2.37 90) (layer F.Fab)
       (effects (font (size 1 1) (thickness 0.15)))
     )
@@
       (net 4 +5V))
     (pad 2 thru_hole circle (at 8.2 -7) (size 2 2) (drill 1) (layers *.Cu *.Mask)
-      (net 22 "Net-(J1-Pad9)"))
+      (net 32 "Net-(R7-Pad1)"))
     (pad A thru_hole circle (at 3.2 7.5) (size 2 2) (drill 1) (layers *.Cu *.Mask)
       (net 30 "Net-(R1-Pad2)"))
@@
   )
   (module Capacitor_THT:C_Disc_D5.1mm_W3.2mm_P5.00mm (layer F.Cu)
-    (at 77 75 180)
+    (at 79.5 75 180)
     (descr "C, Disc series, Radial, pin pitch=5.00mm, , diameter*width=5.1*3.2mm^2, Capacitor, http://www.vishay.com/docs/45233/krseries.pdf")
     (tags "C Disc series Radial pin pitch 5.00mm  diameter 5.1mm width 3.2mm Capacitor")
@@
     )
   )
-  (gr_text v1.1 (at 77 70.5) (layer F.SilkS)
+  (module Resistor_THT:R_Axial_DIN0207_L6.3mm_D2.5mm_P10.16mm_Horizontal (layer F.Cu)
+    (at 82.377 132)
+    (descr "Resistor, Axial_DIN0207 series, Axial, Horizontal, pin pitch=10.16mm, 0.25W = 1/4W, length*diameter=6.3*2.5mm^2, http://cdn-reichelt.de/documents/datenblatt/B400/1_4W%23YAG.pdf")
+    (tags "Resistor Axial_DIN0207 series Axial Horizontal pin pitch 10.16mm 0.25W = 1/4W length 6.3mm diameter 2.5mm")
+    (fp_text reference R7 (at 5.08 -2.37) (layer F.SilkS)
+      (effects (font (size 1 1) (thickness 0.15)))
+    )
+    (fp_text value 1K (at 5.08 2.37) (layer F.Fab)
+      (effects (font (size 1 1) (thickness 0.15)))
+    )
+    (fp_line (start 1.93 -1.25) (end 1.93 1.25) (layer F.Fab) (width 0.1))
+    (fp_line (start 1.93 1.25) (end 8.23 1.25) (layer F.Fab) (width 0.1))
+    (fp_line (start 8.23 1.25) (end 8.23 -1.25) (layer F.Fab) (width 0.1))
+    (fp_line (start 8.23 -1.25) (end 1.93 -1.25) (layer F.Fab) (width 0.1))
+    (fp_line (start 0 0) (end 1.93 0) (layer F.Fab) (width 0.1))
+    (fp_line (start 10.16 0) (end 8.23 0) (layer F.Fab) (width 0.1))
+    (fp_line (start 1.81 -1.37) (end 1.81 1.37) (layer F.SilkS) (width 0.12))
+    (fp_line (start 1.81 1.37) (end 8.35 1.37) (layer F.SilkS) (width 0.12))
+    (fp_line (start 8.35 1.37) (end 8.35 -1.37) (layer F.SilkS) (width 0.12))
+    (fp_line (start 8.35 -1.37) (end 1.81 -1.37) (layer F.SilkS) (width 0.12))
+    (fp_line (start 1.04 0) (end 1.81 0) (layer F.SilkS) (width 0.12))
+    (fp_line (start 9.12 0) (end 8.35 0) (layer F.SilkS) (width 0.12))
+    (fp_line (start -1.05 -1.5) (end -1.05 1.5) (layer F.CrtYd) (width 0.05))
+    (fp_line (start -1.05 1.5) (end 11.21 1.5) (layer F.CrtYd) (width 0.05))
+    (fp_line (start 11.21 1.5) (end 11.21 -1.5) (layer F.CrtYd) (width 0.05))
+    (fp_line (start 11.21 -1.5) (end -1.05 -1.5) (layer F.CrtYd) (width 0.05))
+    (fp_text user %R (at 5.08 0) (layer F.Fab)
+      (effects (font (size 1 1) (thickness 0.15)))
+    )
+    (pad 1 thru_hole circle (at 0 0) (size 1.6 1.6) (drill 0.8) (layers *.Cu *.Mask)
+      (net 32 "Net-(R7-Pad1)"))
+    (pad 2 thru_hole oval (at 10.16 0) (size 1.6 1.6) (drill 0.8) (layers *.Cu *.Mask)
+      (net 22 "Net-(J1-Pad9)"))
+    (model ${KISYS3DMOD}/Resistor_THT.3dshapes/R_Axial_DIN0207_L6.3mm_D2.5mm_P10.16mm_Horizontal.wrl
+      (at (xyz 0 0 0))
+      (scale (xyz 1 1 1))
+      (rotate (xyz 0 0 0))
+    )
+  )
+  (gr_text v1.2 (at 77 70.5) (layer F.SilkS)
     (effects (font (size 1.5 1.5) (thickness 0.15)))
   )
@@
   (gr_line (start 60 60) (end 95 60) (layer Edge.Cuts) (width 0.1))
   (gr_line (start 60 170) (end 60 60) (layer Edge.Cuts) (width 0.1))
+  (segment (start 78 112) (end 78 112) (width 0.25) (layer F.Cu) (net 1))
+  (via (at 78 112) (size 0.8) (drill 0.4) (layers F.Cu B.Cu) (net 1))
+  (segment (start 76 114) (end 78 112) (width 0.25) (layer B.Cu) (net 1))
+  (segment (start 76 137) (end 76 114) (width 0.25) (layer B.Cu) (net 1))
+  (segment (start 88.96 95.12) (end 84.5 99.58) (width 0.25) (layer B.Cu) (net 1))
+  (segment (start 84.5 99.58) (end 84.5 112) (width 0.25) (layer B.Cu) (net 1))
+  (segment (start 84.5 112) (end 84.5 112) (width 0.25) (layer B.Cu) (net 1))
+  (via (at 84.5 112) (size 0.8) (drill 0.4) (layers F.Cu B.Cu) (net 1))
+  (segment (start 78 112) (end 84.5 112) (width 0.25) (layer F.Cu) (net 1))
+  (segment (start 64.799999 157.200001) (end 64 158) (width 0.25) (layer B.Cu) (net 1))
+  (segment (start 74.874999 147.125001) (end 64.799999 157.200001) (width 0.25) (layer B.Cu) (net 1))
+  (segment (start 74.874999 138.125001) (end 74.874999 147.125001) (width 0.25) (layer B.Cu) (net 1))
+  (segment (start 76 137) (end 74.874999 138.125001) (width 0.25) (layer B.Cu) (net 1))
   (segment (start 89 157.7) (end 89 157) (width 0.25) (layer F.Cu) (net 3))
+  (segment (start 88.200001 156.200001) (end 89 157) (width 0.25) (layer B.Cu) (net 3))
+  (segment (start 85.125001 153.125001) (end 88.200001 156.200001) (width 0.25) (layer B.Cu) (net 3))
+  (segment (start 85.125001 138.125001) (end 85.125001 153.125001) (width 0.25) (layer B.Cu) (net 3))
+  (segment (start 84 137) (end 85.125001 138.125001) (width 0.25) (layer B.Cu) (net 3))
+  (segment (start 84 137) (end 86 135) (width 0.25) (layer F.Cu) (net 3))
+  (segment (start 92.88 96.5) (end 91.5 95.12) (width 0.25) (layer B.Cu) (net 3))
+  (segment (start 93 96.5) (end 92.88 96.5) (width 0.25) (layer B.Cu) (net 3))
+  (segment (start 93 128) (end 93 96.5) (width 0.25) (layer B.Cu) (net 3))
+  (segment (start 94 135) (end 94 135) (width 0.25) (layer B.Cu) (net 3))
+  (segment (start 94 129) (end 93 128) (width 0.25) (layer B.Cu) (net 3))
+  (segment (start 94 135) (end 94 129) (width 0.25) (layer B.Cu) (net 3))
+  (via (at 94 135) (size 0.8) (drill 0.4) (layers F.Cu B.Cu) (net 3))
+  (segment (start 86 135) (end 94 135) (width 0.25) (layer F.Cu) (net 3))
   (segment (start 67.54 152) (end 65.54 150) (width 0.25) (layer F.Cu) (net 4))
   (segment (start 75.2 152) (end 67.54 152) (width 0.25) (layer F.Cu) (net 4))
@@
   (segment (start 88.96 92.58) (end 82.814999 98.725001) (width 0.25) (layer B.Cu) (net 21))
   (segment (start 82.725001 98.725001) (end 82.725001 117.774999) (width 0.25) (layer B.Cu) (net 21))
-  (segment (start 93 128) (end 84 137) (width 0.25) (layer B.Cu) (net 3))
-  (segment (start 93 128) (end 93 96.5) (width 0.25) (layer B.Cu) (net 3))
-  (segment (start 92.88 96.5) (end 91.5 95.12) (width 0.25) (layer B.Cu) (net 3))
-  (segment (start 93 96.5) (end 92.88 96.5) (width 0.25) (layer B.Cu) (net 3))
-  (segment (start 78 112) (end 78 112) (width 0.25) (layer F.Cu) (net 1))
-  (via (at 78 112) (size 0.8) (drill 0.4) (layers F.Cu B.Cu) (net 1))
-  (segment (start 76 114) (end 78 112) (width 0.25) (layer B.Cu) (net 1))
-  (segment (start 76 137) (end 76 114) (width 0.25) (layer B.Cu) (net 1))
-  (segment (start 88.96 95.12) (end 84.5 99.58) (width 0.25) (layer B.Cu) (net 1))
-  (segment (start 84.5 99.58) (end 84.5 112) (width 0.25) (layer B.Cu) (net 1))
-  (segment (start 84.5 112) (end 84.5 112) (width 0.25) (layer B.Cu) (net 1))
-  (via (at 84.5 112) (size 0.8) (drill 0.4) (layers F.Cu B.Cu) (net 1))
-  (segment (start 78 112) (end 84.5 112) (width 0.25) (layer F.Cu) (net 1))
-  (segment (start 64.799999 157.200001) (end 64 158) (width 0.25) (layer B.Cu) (net 1))
-  (segment (start 74.874999 147.125001) (end 64.799999 157.200001) (width 0.25) (layer B.Cu) (net 1))
-  (segment (start 74.874999 138.125001) (end 74.874999 147.125001) (width 0.25) (layer B.Cu) (net 1))
-  (segment (start 76 137) (end 74.874999 138.125001) (width 0.25) (layer B.Cu) (net 1))
-  (segment (start 88.200001 156.200001) (end 89 157) (width 0.25) (layer B.Cu) (net 3))
-  (segment (start 85.125001 153.125001) (end 88.200001 156.200001) (width 0.25) (layer B.Cu) (net 3))
-  (segment (start 85.125001 138.125001) (end 85.125001 153.125001) (width 0.25) (layer B.Cu) (net 3))
-  (segment (start 84 137) (end 85.125001 138.125001) (width 0.25) (layer B.Cu) (net 3))
-  (segment (start 80.2 136.8) (end 80.2 151) (width 0.25) (layer B.Cu) (net 22))
-  (segment (start 88 129) (end 80.2 136.8) (width 0.25) (layer B.Cu) (net 22))
   (segment (start 92.54999 98.70999) (end 92.54999 124.45001) (width 0.25) (layer B.Cu) (net 22))
   (segment (start 91.5 97.66) (end 92.54999 98.70999) (width 0.25) (layer B.Cu) (net 22))
-  (segment (start 92.54999 124.45001) (end 88 129) (width 0.25) (layer B.Cu) (net 22))
+  (segment (start 92.537 132) (end 92.537 124.537) (width 0.25) (layer B.Cu) (net 22))
   (segment (start 84.96 116.54) (end 85 116.5) (width 0.25) (layer F.Cu) (net 23))
   (segment (start 79.62 116.54) (end 84.96 116.54) (width 0.25) (layer F.Cu) (net 23))
@@
   (segment (start 84 147.16) (end 81.674999 149.485001) (width 0.25) (layer B.Cu) (net 31))
   (segment (start 84 147.16) (end 89 147.16) (width 0.25) (layer F.Cu) (net 31))
+  (segment (start 80.2 134.177) (end 82.377 132) (width 0.25) (layer B.Cu) (net 32))
+  (segment (start 80.2 151) (end 80.2 134.177) (width 0.25) (layer B.Cu) (net 32))
   (zone (net 2) (net_name GND) (layer F.Cu) (hatch edge 0.508)
     (connect_pads (clearance 0.508))
